File: projects/Bootcamp_elec42/Bootcamp_elec42.kicad_sch (KiCad schematic)
At the start: 0 parts

Commit message: [ADD] Symbols finished, schematic done
Parts:
- added ATmega328P-AU1: U1, symbol MCU_Atmel_42ChipsPro_Mini:MCU_Atmega328P_AU
- added C1, C2: 12pF, symbol MCU_Atmel_42ChipsPro_Mini:C
- added C3, C4, C7: 100nF, symbol MCU_Atmel_42ChipsPro_Mini:C
- added C6: 1uF, symbol MCU_Atmel_42ChipsPro_Mini:C
- added D1: Green, symbol MCU_Atmel_42ChipsPro_Mini:D
- added D2: Red, symbol MCU_Atmel_42ChipsPro_Mini:D
- added J1: ~, symbol MCU_Atmel_42ChipsPro_Mini:J1
- added J2: ~, symbol MCU_Atmel_42ChipsPro_Mini:J2
- added J3: ~, symbol MCU_Atmel_42ChipsPro_Mini:J3
- added R1: 330, symbol MCU_Atmel_42ChipsPro_Mini:R
- added R2, R3: 10K, symbol MCU_Atmel_42ChipsPro_Mini:R
- added SW1: SW_Push, symbol MCU_Atmel_42ChipsPro_Mini:SW
- added Y1: ~, symbol MCU_Atmel_42ChipsPro_Mini:Y
Connections:
- new net: C4.2, SW1.1
- new net: ATmega328P-AU1.8 ((PCINT7/XTAL2/TOSC2)_PB7), C1.1, Y1.1
- new net: ATmega328P-AU1.7 ((PCINT6/XTAL1/TOSC1)_PB6), C2.1, Y1.3
- new net: D1.1, R1.2
- new net: D2.2, R2.1
- new net: ATmega328P-AU1.20 (AREF), C3.1
- new net A0: ATmega328P-AU1.23 ((ADC0/PCINT8)_PC0), J2.8
- new net A1: ATmega328P-AU1.24 ((ADC1/PCINT9)_PC1), J2.7
- new net A2: ATmega328P-AU1.25 ((ADC2/PCINT10)_PC2), J2.6
- new net A3: ATmega328P-AU1.26 ((ADC3/PCINT11)_PC3), J2.5
- new net A4: ATmega328P-AU1.27 ((ADC4/SDA/PCINT12)_PC4)
- new net A5: ATmega328P-AU1.28 ((ADC5/SCL/PCINT13)_PC5)
- new net A6: ATmega328P-AU1.19 (ADC6)
- new net A7: ATmega328P-AU1.22 (ADC7)
- new net D10: ATmega328P-AU1.14 ((PCINT2/SS/OC1B)_PB2), J2.12
- new net D2: ATmega328P-AU1.32 ((INT0/PCINT18)_PD2), J1.8
- new net D3: ATmega328P-AU1.1 ((PCINT19/OC2B/INT)_PD3), J1.7
- new net D4: ATmega328P-AU1.2 ((PCINT20/XCK/T0)_PD4), J1.6
- new net D5: ATmega328P-AU1.9 ((PCINT21/OC0B/T1)_PD5), J1.5
- new net D6: ATmega328P-AU1.10 ((PCINT22/OC0A/ATN0)_PD6), J1.4
- new net D7: ATmega328P-AU1.11 ((PCINT23/AIN1)_PD7), J1.3
- new net D8: ATmega328P-AU1.12 ((PCINT0/CLKO/ICP1)_PB0), J1.2
- new net D9: ATmega328P-AU1.13 ((PCINT1/OC1A)_PB1), J1.1
- new net DTR: ATmega328P-AU1.29 ((RESET/PCINT14)_PC6), J1.10, J2.3, J3.1, R3.1, SW1.2
- new net GND: ATmega328P-AU1.3 (GND_1), C1.2, C2.2, C4.1, C6.2, C7.2, D1.2, J1.9, J2.2, J3.5, J3.6, R2.2, Y1.2, Y1.4
- new net MISO: ATmega328P-AU1.16 ((PCINT4/MISO)_PB4), J2.10
- new net MOSI: ATmega328P-AU1.15 ((PCINT3/OC2A/MOSI)_PB3), J2.11
- new net RXI: ATmega328P-AU1.30 ((RXD/PCINT16)_PD0), J1.11, J3.3
- new net SCK: ATmega328P-AU1.17 ((SCK/PCINT5)_PB5), J2.9, R1.1
- new net TXO: ATmega328P-AU1.31 ((TXD/PCINT17)_PD1), J1.12, J3.2
- new net VCC: ATmega328P-AU1.18 (AVCC), ATmega328P-AU1.4 (VCC_1), C3.2, C6.1, C7.1, D2.1, J2.1, J2.4, J3.4, R3.2
- no-connect marks 0 -> 5
Other:
- note added: "Activity"
- note added: "Power"
- note added: "Reset"

Commit message: SMD Done~
Parts:
- ATmega328P-AU1: footprint (none) -> Footprint:ATMEGA328P; LCSC Part Number (none) -> C14877
- C1, C2: footprint (none) -> Footprint:CR_Generic; LCSC Part Number (none) -> C38523
- C3, C4, C7: footprint (none) -> Footprint:CR_Generic; LCSC Part Number (none) -> C14663
- C6: footprint (none) -> Footprint:CR_Generic; LCSC Part Number (none) -> C15849
- D1: footprint (none) -> Footprint:LED_generic; LCSC Part Number (none) -> C916074
- D2: footprint (none) -> Footprint:LED_generic; LCSC Part Number (none) -> C965799
- J1, J2: footprint (none) -> Footprint:PinHeader_12
- J3: footprint (none) -> Footprint:PinHeader_6
- R1: footprint (none) -> Footprint:CR_Generic; LCSC Part Number (none) -> C23138
- R2, R3: footprint (none) -> Footprint:CR_Generic; LCSC Part Number (none) -> C98220
- SW1: footprint (none) -> Footprint:SW_B3U1000P; LCSC Part Number (none) -> C231329
- Y1: footprint (none) -> Footprint:Crystal_YSX321SL; LCSC Part Number (none) -> C13738
Other:
- moved on the sheet: ATmega328P-AU1, C6, C7, D2, J2, J3, R2

Commit message: Files needed
Changed lines of the file:
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@@
 	(symbol
 		(lib_id "MCU_Atmel_42ChipsPro_Mini:GND")
-		(at 278.13 157.48 0)
+		(at 273.05 157.48 0)
 		(unit 1)
 		(exclude_from_sim yes)
@@
 		(fields_autoplaced yes)
 		(property "Reference" "#GND00"
-			(at 280.67 155.5749 0)
+			(at 275.59 155.5749 0)
 			(effects
 				(font
@@
 		)
 		(property "Value" "GND"
-			(at 280.67 158.1149 0)
+			(at 275.59 158.1149 0)
 			(effects
 				(font
@@
 		)
 		(property "Footprint" ""
-			(at 278.13 157.48 0)
-			(effects
-				(font
-					(size 1.27 1.27)
-				)
-				(hide yes)
-			)
-		)
-		(property "Datasheet" ""
-			(at 278.13 157.48 0)
+			(at 273.05 157.48 0)
+			(effects
+				(font
+					(size 1.27 1.27)
+				)
+				(hide yes)
+			)
+		)
+		(property "Datasheet" ""
+			(at 273.05 157.48 0)
 			(effects
 				(font
@@
 		)
 		(property "Description" ""
-			(at 278.13 157.48 0)
+			(at 273.05 157.48 0)
 			(effects
 				(font
@@
 	(symbol
 		(lib_id "MCU_Atmel_42ChipsPro_Mini:Power_output")
-		(at 278.13 161.29 0)
+		(at 273.05 161.29 0)
 		(unit 1)
 		(exclude_from_sim no)
@@
 		(fields_autoplaced yes)
 		(property "Reference" "#PO02"
-			(at 280.67 162.5599 0)
+			(at 275.59 162.5599 0)
 			(effects
 				(font
@@
 		)
 		(property "Value" "~"
-			(at 280.67 165.0999 0)
+			(at 275.59 165.0999 0)
 			(effects
 				(font
@@
 		)
 		(property "Footprint" ""
-			(at 278.13 161.29 0)
-			(effects
-				(font
-					(size 1.27 1.27)
-				)
-				(hide yes)
-			)
-		)
-		(property "Datasheet" ""
-			(at 278.13 161.29 0)
+			(at 273.05 161.29 0)
+			(effects
+				(font
+					(size 1.27 1.27)
+				)
+				(hide yes)
+			)
+		)
+		(property "Datasheet" ""
+			(at 273.05 161.29 0)
 			(effects
 				(font
@@
 		)
 		(property "Description" ""
-			(at 278.13 161.29 0)
+			(at 273.05 161.29 0)
 			(effects
 				(font
@@
 	(symbol
 		(lib_id "MCU_Atmel_42ChipsPro_Mini:Power_output")
-		(at 264.16 161.29 0)
+		(at 259.08 161.29 0)
 		(unit 1)
 		(exclude_from_sim no)
@@
 		(fields_autoplaced yes)
 		(property "Reference" "#PO01"
-			(at 266.7 162.5599 0)
+			(at 261.62 162.5599 0)
 			(effects
 				(font
@@
 		)
 		(property "Value" "~"
-			(at 266.7 165.0999 0)
+			(at 261.62 165.0999 0)
 			(effects
 				(font
@@
 		)
 		(property "Footprint" ""
-			(at 264.16 161.29 0)
-			(effects
-				(font
-					(size 1.27 1.27)
-				)
-				(hide yes)
-			)
-		)
-		(property "Datasheet" ""
-			(at 264.16 161.29 0)
+			(at 259.08 161.29 0)
+			(effects
+				(font
+					(size 1.27 1.27)
+				)
+				(hide yes)
+			)
+		)
+		(property "Datasheet" ""
+			(at 259.08 161.29 0)
 			(effects
 				(font
@@
 		)
 		(property "Description" ""
-			(at 264.16 161.29 0)
+			(at 259.08 161.29 0)
 			(effects
 				(font
@@
 	(symbol
 		(lib_id "MCU_Atmel_42ChipsPro_Mini:VCC")
-		(at 264.16 157.48 0)
+		(at 259.08 157.48 0)
 		(unit 1)
 		(exclude_from_sim yes)
@@
 		(fields_autoplaced yes)
 		(property "Reference" "#VCC00"
-			(at 266.7 155.5749 0)
+			(at 261.62 155.5749 0)
 			(effects
 				(font
@@
 		)
 		(property "Value" "VCC"
-			(at 266.7 158.1149 0)
+			(at 261.62 158.1149 0)
 			(effects
 				(font
@@
 		)
 		(property "Footprint" ""
-			(at 264.16 157.48 0)
-			(effects
-				(font
-					(size 1.27 1.27)
-				)
-				(hide yes)
-			)
-		)
-		(property "Datasheet" ""
-			(at 264.16 157.48 0)
+			(at 259.08 157.48 0)
+			(effects
+				(font
+					(size 1.27 1.27)
+				)
+				(hide yes)
+			)
+		)
+		(property "Datasheet" ""
+			(at 259.08 157.48 0)
 			(effects
 				(font
@@
 		)
 		(property "Description" ""
-			(at 264.16 157.48 0)
-			(effects
-				(font
+			(at 259.08 157.48 0)
+			(effects
+				(font
